File: 回路/QX20CTRLV2/QX20CTRLV2.kicad_pcb (KiCad board)
At the start: 2 copper layers, 70 x 45 mm, 29 parts, among them J1 VH_CAN, J2 VH_CAN, J3 VH_SRV1, J4 VH_SRV2, J5 USART, J6 I2C, SW1 SKRP, SW2 SW_SPDT, SW3 SKRP, SW4 SKRP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

Commit message: QX20CTRLV2 ガーバーデータ
Parts:
- C1, C2, C6, D1, R3: moved to B.Cu
- moved D2 26.0 mm to (112.0, 55.5), turned to 90 degrees
- moved D3 17.0 mm to (150.0, 70.5), turned to 0 degrees
- moved REF** 16.3 mm to (145.5, 60.5)
- moved D1 14.5 mm to (135.0, 89.2)
- moved J5 12.8 mm to (151.0, 81.0)
- moved C2 12.1 mm to (151.5, 86.0), turned to 0 degrees
- moved R2 9.69 mm to (138.5, 54.0), turned to 180 degrees
- moved U3 8.51 mm to (142.5, 70.5)
- moved C6 6.49 mm to (141.5, 70.5), turned to 0 degrees
- moved R3 5.93 mm to (156.0, 64.2), turned to 270 degrees
- moved C1 2.01 mm to (139.5, 89.0)
- moved SW3 1.50 mm to (121.0, 91.0)
- moved SW1 1.00 mm to (121.5, 82.0)
Routing:
- net VIN: track 240.7 -> 2.50 mm
- net GND: track 67.2 -> 37.7 mm, vias 5 -> 2
- net 3.3V: track 103.4 -> 125.6 mm, vias 3 -> 2
- net Net-(D2-Pad2): track 3.50 -> 25.0 mm
- net USART_TX: track 6.14 -> 20.0 mm
- net USART_RX: track 6.23 -> 20.0 mm
- net CAN_TX: track 21.4 -> 8.03 mm
- net Net-(R2-Pad1): track 5.94 -> 17.2 mm
- net CAN_RX: track 14.7 -> 7.45 mm
- net CANL: track 43.1 -> 37.0 mm
- net CANH: track 41.0 -> 43.3 mm
- net PWM2: track 17.9 -> 15.9 mm
- net PWM1: track 27.7 -> 25.8 mm
- net Net-(SW3-Pad1): track 18.3 -> 19.3 mm
- added copper zone on B.Cu, net VIN
Other:
- net class 3.3V: via_dia 1.15 -> 1.4
- net class Default: via_dia 1.15 -> 1.4
- net class Power: via_dia 1.15 -> 1.4
