File: 回路/QX20CTRLV3/QX20CTRLV3.sch (KiCad schematic (older format))
At the start: 21 parts, among them J1 VH_CAN, J2 VH_CAN, J3 VH_SRV1, J4 VH_SRV2, J5 USART, J6 I2C, J7 Conn_01x05, SW2 SW_SPDT, U1 BP5293-33, U2 STM32F303K8Tx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

Commit message: QX20CTRLV3発注仕様
Parts:
- added R3, R4: 0, Resistor_SMD:R_1206_3216Metric_Pad1.42x1.75mm_HandSolder, symbol Device:R_Small
- J5: footprint Connector_PinHeader_2.54mm:PinHeader_1x03_P2.54mm_Vertical -> Connector_JST:JST_XH_B3B-XH-A_1x03_P2.50mm_Vertical
- J6: footprint Connector_PinHeader_2.54mm:PinHeader_1x04_P2.54mm_Vertical -> Connector_JST:JST_XH_B4B-XH-A_1x04_P2.50mm_Vertical
- J7: footprint Connector_PinHeader_2.54mm:PinHeader_1x05_P2.54mm_Vertical -> Connector_JST:JST_XH_B5B-XH-A_1x05_P2.50mm_Vertical
Connections:
- net CANH: now also D3.1 (K); no longer D3.2 (K)
- net CANL: now also D3.2 (K); no longer D3.1 (K)
- net PWM1: now also R3.2; no longer J3.1 (Pin_1)
- net PWM2: now also R4.2; no longer J4.1 (Pin_1)
- new net: J3.1 (Pin_1), R3.1
- new net: J4.1 (Pin_1), R4.1
Changed lines of the file:
@@
 F 0 "J6" H 918 4925 50  0000 C CNN
 F 1 "I2C" H 918 5016 50  0000 C CNN
-F 2 "Connector_PinHeader_2.54mm:PinHeader_1x04_P2.54mm_Vertical" H 1000 5350 50  0001 C CNN
+F 2 "Connector_JST:JST_XH_B4B-XH-A_1x04_P2.50mm_Vertical" H 1000 5350 50  0001 C CNN
 F 3 "~" H 1000 5350 50  0001 C CNN
 	1    1000 5350
@@
 F 0 "J5" H 918 4025 50  0000 C CNN
 F 1 "USART" H 918 4116 50  0000 C CNN
-F 2 "Connector_PinHeader_2.54mm:PinHeader_1x03_P2.54mm_Vertical" H 1000 4350 50  0001 C CNN
+F 2 "Connector_JST:JST_XH_B3B-XH-A_1x03_P2.50mm_Vertical" H 1000 4350 50  0001 C CNN
 F 3 "~" H 1000 4350 50  0001 C CNN
 	1    1000 4350
@@
 NoConn ~ 5850 3850
 NoConn ~ 5850 3750
-Wire Wire Line
-	1200 2700 2050 2700
-Wire Wire Line
-	1200 3250 2050 3250
 Wire Wire Line
 	1200 4250 1650 4250
@@
 F 0 "J7" H 7330 2992 50  0000 L CNN
 F 1 "Conn_01x05" H 7330 2901 50  0000 L CNN
-F 2 "Connector_PinHeader_2.54mm:PinHeader_1x05_P2.54mm_Vertical" H 7250 2950 50  0001 C CNN
+F 2 "Connector_JST:JST_XH_B5B-XH-A_1x05_P2.50mm_Vertical" H 7250 2950 50  0001 C CNN
 F 3 "~" H 7250 2950 50  0001 C CNN
 	1    7250 2950
@@
 	1600 1400 1850 1400
 Wire Wire Line
-	9250 5400 9850 5400
-Wire Wire Line
-	9250 5200 10050 5200
-Wire Wire Line
 	9950 5900 8850 5900
 $Comp
@@
 	1    0    0    -1
 $EndComp
-Wire Wire Line
-	9850 5500 9850 5400
-Connection ~ 9850 5400
-Wire Wire Line
-	9850 5400 10150 5400
-Wire Wire Line
-	10050 5500 10050 5200
-Connection ~ 10050 5200
-Wire Wire Line
-	10050 5200 10150 5200
+$Comp
+L Device:R_Small R4
+U 1 1 5E6FB923
+P 1850 3250
+F 0 "R4" V 1950 3250 50  0000 C CNN
+F 1 "0" V 2050 3250 50  0000 C CNN
+F 2 "Resistor_SMD:R_1206_3216Metric_Pad1.42x1.75mm_HandSolder" H 1850 3250 50  0001 C CNN
+F 3 "" H 1850 3250 50  0001 C CNN
+	1    1850 3250
+	0    -1   -1   0
+$EndComp
+$Comp
+L Device:R_Small R3
+U 1 1 5E6FF84D
+P 1850 2700
+F 0 "R3" V 1950 2700 50  0000 C CNN
+F 1 "0" V 2050 2700 50  0000 C CNN
+F 2 "Resistor_SMD:R_1206_3216Metric_Pad1.42x1.75mm_HandSolder" H 1850 2700 50  0001 C CNN
+F 3 "" H 1850 2700 50  0001 C CNN
+	1    1850 2700
+	0    -1   -1   0
+$EndComp
+Wire Wire Line
+	2050 2700 1950 2700
+Wire Wire Line
+	1750 2700 1200 2700
+Wire Wire Line
+	1200 3250 1750 3250
+Wire Wire Line
+	1950 3250 2050 3250
+Wire Wire Line
+	9250 5400 10050 5400
+Wire Wire Line
+	9250 5200 9850 5200
+Wire Wire Line
+	10050 5400 10050 5500
+Connection ~ 10050 5400
+Wire Wire Line
+	10050 5400 10150 5400
+Wire Wire Line
+	9850 5500 9850 5200
+Connection ~ 9850 5200
+Wire Wire Line
+	9850 5200 10150 5200
 $EndSCHEMATC
