File: 回路/QX20CVT6B8V1/QX20CVT6B8V1.kicad_pcb (KiCad board)
At the start: 2 copper layers, 40 x 27.5 mm, 21 parts, among them J1 VH_VIN, J2 VH_OUT, Q1 Q_HP8K22, U1 L6726A

Commit message: QX20CTRLV3
たまっていた分を更新...
Parts:
- added Q2: RS1E150GN, Package_SON:VSONP-8-1EP_5x6_P1.27mm, F.Cu at (122.6, 122.5)
- C1, C3, C4, C5, C8, C9: footprint Capacitor_SMD:C_1206_3216Metric -> Capacitor_SMD:C_1206_3216Metric_Pad1.42x1.75mm_HandSolder
- C2, C6: footprint Capacitor_SMD:C_0603_1608Metric_Pad1.05x0.95mm_HandSolder -> Capacitor_SMD:C_1206_3216Metric_Pad1.42x1.75mm_HandSolder
- C7, D1: moved to F.Cu
- Q1: value Q_HP8K22 -> RS1E150GN; footprint QX20CVT6B8V1:HSOP8-AD_5x6_P1.27mm -> Package_SON:VSONP-8-1EP_5x6_P1.27mm
- R1, R5, R6: footprint Resistor_SMD:R_0603_1608Metric_Pad1.05x0.95mm_HandSolder -> Resistor_SMD:R_1206_3216Metric_Pad1.42x1.75mm_HandSolder
- R2: value 330 -> 340; footprint Resistor_SMD:R_0603_1608Metric_Pad1.05x0.95mm_HandSolder -> Resistor_SMD:R_1206_3216Metric_Pad1.42x1.75mm_HandSolder; moved to F.Cu
- R3, R4: footprint Resistor_SMD:R_0603_1608Metric_Pad1.05x0.95mm_HandSolder -> Resistor_SMD:R_1206_3216Metric_Pad1.42x1.75mm_HandSolder; moved to F.Cu
- moved R5 56.0 mm to (114.0, 127.0), turned to 180 degrees
- moved R6 35.3 mm to (128.0, 120.0), turned to 90 degrees
- moved C8 31.3 mm to (122.0, 113.5), turned to 0 degrees
- moved C6 28.8 mm to (128.0, 114.0)
- moved C9 28.5 mm to (122.0, 110.5), turned to 0 degrees
- moved R3 27.9 mm to (111.0, 117.0), turned to 90 degrees
- moved R2 19.8 mm to (108.0, 117.0)
- moved R4 19.0 mm to (120.0, 103.5), turned to 270 degrees
- moved J1 15.0 mm to (110.4, 107.4)
- moved J2 14.6 mm to (144.7, 110.4), turned to 90 degrees
- moved C4 13.5 mm to (102.0, 125.5), turned to 90 degrees
- moved U1 13.0 mm to (107.0, 124.5), turned to 90 degrees
- moved D1 10.1 mm to (123.5, 103.2), turned to 90 degrees
- moved L1 9.71 mm to (137.0, 120.5), turned to 90 degrees
- moved C5 9.15 mm to (122.0, 116.5)
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Connections:
- Q1 pad 1: Net-(Q1-Pad1) -> /PHASE
- Q1 pad 2: VIN -> Net-(Q1-Pad2)
- Q1 pad 3: GNDA -> VIN
- R5 pad 1: Net-(Q1-Pad1) -> Net-(Q1-Pad2)
Other:
- board size 40 x 27.5 mm -> 50 x 30 mm
- board text added: "IN 10-15V OUT 6V 8A"
