File: 回路/QX20CVT6B8V1/QX20CVT6B8V1.sch (KiCad schematic (older format))
At the start: 21 parts, among them J1 VH_VIN, J2 VH_OUT, Q1 Q_HP8K22, U1 L6726A

Commit message: QX20CTRLV3
たまっていた分を更新...
Parts:
- removed Q1: Q_HP8K22, QX20CVT6B8V1:HSOP8-AD_5x6_P1.27mm, symbol QX20CVT6B8:Q_HP8K22
- added Q1, Q2: RS1E150GN, Package_SON:VSONP-8-1EP_5x6_P1.27mm, symbol Device:Q_NMOS_SGD
- C1, C3, C4, C5, C8, C9: footprint Capacitor_SMD:C_1206_3216Metric -> Capacitor_SMD:C_1206_3216Metric_Pad1.42x1.75mm_HandSolder
- C2, C6: footprint Capacitor_SMD:C_0603_1608Metric_Pad1.05x0.95mm_HandSolder -> Capacitor_SMD:C_1206_3216Metric_Pad1.42x1.75mm_HandSolder
- R1, R3: footprint Resistor_SMD:R_0603_1608Metric_Pad1.05x0.95mm_HandSolder -> Resistor_SMD:R_1206_3216Metric_Pad1.42x1.75mm_HandSolder
- R2: value 330 -> 340; footprint Resistor_SMD:R_0603_1608Metric_Pad1.05x0.95mm_HandSolder -> Resistor_SMD:R_1206_3216Metric_Pad1.42x1.75mm_HandSolder
Connections:
- net GNDA: now also Q2.1 (S)
- net LGATE: now also Q2.2 (G)
- net PHASE: now also Q1.1 (S), Q2.3 (D)
- net VIN: now also Q1.3 (D)
- net at R5.1: now also Q1.2 (G)
Other:
- moved on the sheet: R5
